File: hardware/oct05-mincaps/ria-backplane-mincaps/pcb/ria.kicad_sch (KiCad schematic)
At the start: 69 parts

Commit message: value engineer capacitor sourcing and use available regulator
Parts:
- ESP-C3: footprint ria:ESP-C3 -> ria:C_0805_2012Metric; LCSC C15849 -> C28323; MPN (none) -> CL21B105KBFNNNE; Manufacturer (none) -> Samsung Electro-Mechanics; Supplier Part Number (none) -> C28323
- MOTOR1-C2: footprint ria:MOTOR1-C2 -> ria:C_0805_2012Metric; LCSC C59782 -> C28323; MPN CL10B105KO8NNNC -> CL21B105KBFNNNE; Manufacturer (none) -> Samsung Electro-Mechanics; Supplier Part Number (none) -> C28323
- MOTOR1-C5: value 10uF -> 22uF; footprint ria:MOTOR1-C5 -> ria:C_1206_3216Metric; LCSC C39232 -> C12891; MPN (none) -> CL31A226KAHNNNE; Manufacturer (none) -> Samsung Electro-Mechanics; Supplier Part Number (none) -> C12891
- MOTOR2-C2: footprint ria:MOTOR2-C2 -> ria:C_0805_2012Metric; LCSC C59782 -> C28323; MPN CL10B105KO8NNNC -> CL21B105KBFNNNE; Manufacturer (none) -> Samsung Electro-Mechanics; Supplier Part Number (none) -> C28323
- MOTOR2-C5: value 10uF -> 22uF; footprint ria:MOTOR2-C5 -> ria:C_1206_3216Metric; LCSC C39232 -> C12891; MPN (none) -> CL31A226KAHNNNE; Manufacturer (none) -> Samsung Electro-Mechanics; Supplier Part Number (none) -> C12891
- MOTOR3-C2: footprint ria:MOTOR3-C2 -> ria:C_0805_2012Metric; LCSC C59782 -> C28323; MPN CL10B105KO8NNNC -> CL21B105KBFNNNE; Manufacturer (none) -> Samsung Electro-Mechanics; Supplier Part Number (none) -> C28323
- MOTOR3-C5: value 10uF -> 22uF; footprint ria:MOTOR3-C5 -> ria:C_1206_3216Metric; LCSC C39232 -> C12891; MPN (none) -> CL31A226KAHNNNE; Manufacturer (none) -> Samsung Electro-Mechanics; Supplier Part Number (none) -> C12891
- MOTOR4-C2: footprint ria:MOTOR4-C2 -> ria:C_0805_2012Metric; LCSC C59782 -> C28323; MPN CL10B105KO8NNNC -> CL21B105KBFNNNE; Manufacturer (none) -> Samsung Electro-Mechanics; Supplier Part Number (none) -> C28323
- MOTOR4-C5: value 10uF -> 22uF; footprint ria:MOTOR4-C5 -> ria:C_1206_3216Metric; LCSC C39232 -> C12891; MPN (none) -> CL31A226KAHNNNE; Manufacturer (none) -> Samsung Electro-Mechanics; Supplier Part Number (none) -> C12891
- POWER-U1: value AP63300WU-7 -> AP63301WU-7; LCSC C2158012 -> C2158003; MPN AP63300WU-7 -> AP63301WU-7; Manufacturer (none) -> Diodes Incorporated; Supplier Part Number (none) -> C2158003
