File: pcb/ria.kicad_pcb (KiCad board)
At the start: 4 copper layers, 50 x 65 mm, 104 parts

Commit message: remove obsolete pcb copies and generated documentation
Parts:
- removed ESP-C2: 100nF, ria:ESP-C2
- removed IMU-R1, IMU-R2: 4.7kΩ, ria:R_0603_1608Metric
- removed MOTOR1-C10, MOTOR2-C10, MOTOR3-C10, MOTOR4-C10, SENSE-C1: 100nF, ria:C_0603_1608Metric
- removed MOTOR1-C11, MOTOR1-C12, MOTOR2-C11, MOTOR2-C12, MOTOR3-C11, MOTOR3-C12, MOTOR4-C11, MOTOR4-C12: 22pF, ria:C_0603_1608Metric
- removed MOTOR1-C7, MOTOR2-C7, MOTOR3-C7, MOTOR4-C7: 47nF, ria:C_0603_1608Metric
- removed MOTOR1-C8, MOTOR2-C8, MOTOR3-C8, MOTOR4-C8: 22uF, ria:C_0805_2012Metric
- removed MOTOR1-R1, MOTOR2-R1, MOTOR3-R1, MOTOR4-R1: 47kΩ, ria:R_0603_1608Metric
- removed MOTOR1-R2, MOTOR2-R2, MOTOR3-R2, MOTOR4-R2: 22Ω, ria:R_0603_1608Metric
- removed MOTOR1-R3, MOTOR2-R3, MOTOR3-R3, MOTOR4-R3: 5.1kΩ, ria:R_0603_1608Metric
- removed MOTOR1-R4, MOTOR1-R5, MOTOR2-R4, MOTOR2-R5, MOTOR3-R4, MOTOR3-R5, MOTOR4-R4, MOTOR4-R5: 330Ω, ria:R_0603_1608Metric
- removed POWER-C2: 100nF, ria:POWER-C2
- removed SENSE-R1: 100kΩ, ria:R_0603_1608Metric
- removed SENSE-R2: 20kΩ, ria:R_0603_1608Metric
- removed USB-C1: 100nF, ria:USB-C1
- added ENC-J1: ENC-J1, ria:ENC-J1, F.Cu at (78.5, 103.0)
- added ENC-J2: ENC-J2, ria:ENC-J2, F.Cu at (78.5, 114.5)
- added ENC-J3: ENC-J3, ria:ENC-J3, F.Cu at (121.5, 103.0)
- added ENC-J4: ENC-J4, ria:ENC-J4, F.Cu at (121.5, 114.5)
- added ENC-RC0: 4.7kΩ, ria:ENC-RC0, F.Cu at (82.5, 103.5)
- added ENC-RC1: 4.7kΩ, ria:ENC-RC1, F.Cu at (82.5, 114.0)
- added ENC-RC2: 4.7kΩ, ria:ENC-RC2, F.Cu at (117.5, 103.5)
- added ENC-RC3: 4.7kΩ, ria:ENC-RC3, F.Cu at (117.5, 114.0)
- added ENC-RD0: 4.7kΩ, ria:ENC-RD0, F.Cu at (82.5, 100.0)
- added ENC-RD1: 4.7kΩ, ria:ENC-RD1, F.Cu at (82.5, 110.5)
- added ENC-RD2: 4.7kΩ, ria:ENC-RD2, F.Cu at (117.5, 100.0)
- added ENC-RD3: 4.7kΩ, ria:ENC-RD3, F.Cu at (117.5, 110.5)
- added MOTOR-R2: 10kΩ, ria:MOTOR-RS, F.Cu at (82.5, 97.5)
- ESP-C3: footprint ria:ESP-C3 -> ria:C_0805_2012Metric
- MOTOR1-C2, MOTOR2-C2, MOTOR3-C2, MOTOR4-C2: footprint ria:C_0603_1608Metric -> ria:C_0805_2012Metric
- MOTOR1-C3: footprint ria:C_0603_1608Metric -> ria:MOTOR1-C3
- MOTOR1-C5, MOTOR2-C5, MOTOR3-C5, MOTOR4-C5: value 10uF -> 22uF
- MOTOR1-C6: value 1uF -> 4.7uF; footprint ria:C_0805_2012Metric -> ria:MOTOR1-C6
- MOTOR1-U1, MOTOR2-U1, MOTOR3-U1, MOTOR4-U1: value DRV8316CTRGFR -> SS6343M-QF-TP; footprint ria:DRV8316CTRGFR -> ria:SS6343M-QF-TP
- MOTOR2-C3: footprint ria:C_0603_1608Metric -> ria:MOTOR2-C3
- MOTOR2-C6: value 1uF -> 4.7uF; footprint ria:C_0805_2012Metric -> ria:MOTOR2-C6
- MOTOR3-C3: footprint ria:C_0603_1608Metric -> ria:MOTOR3-C3
- MOTOR3-C6: value 1uF -> 4.7uF; footprint ria:C_0805_2012Metric -> ria:MOTOR3-C6
- MOTOR4-C3: footprint ria:C_0603_1608Metric -> ria:MOTOR4-C3
- MOTOR4-C6: value 1uF -> 4.7uF; footprint ria:C_0805_2012Metric -> ria:MOTOR4-C6
- POWER-J1: value XT60PB-M.G.Y -> XT60PW-M
- POWER-U1: value AP63300WU-7 -> AP63301WU-7
- moved POWER-D1 20.4 mm to (95.5, 123.6), turned to -90 degrees
- moved POWER-D2 20.4 mm to (104.5, 123.6)
- moved MOTOR4-C2 10.7 mm to (109.8, 117.7)
- moved MOTOR2-C2 10.3 mm to (107.1, 102.4), turned to 180 degrees
- moved MOTOR1-C2 10.00 mm to (85.1, 102.4), turned to 180 degrees
- moved MOTOR3-C2 8.84 mm to (90.4, 126.6), turned to -90 degrees
- moved MOTOR4-C3 8.45 mm to (111.2, 125.6), turned to 90 degrees
- moved MOTOR3-C3 6.65 mm to (89.8, 117.7), turned to -90 degrees
- moved POWER-J1 4.50 mm to (83.4, 75.7), turned to -90 degrees
- moved MOTOR1-C5 4.10 mm to (89.0, 109.0), turned to 180 degrees
- moved MOTOR2-C5 4.10 mm to (111.0, 109.0), turned to 180 degrees
- moved MOTOR3-C5 3.23 mm to (91.0, 113.5), turned to 180 degrees
- moved MOTOR3-C6 2.98 mm to (92.2, 125.6), turned to 90 degrees
- moved MOTOR4-C6 2.92 mm to (107.8, 117.7), turned to -90 degrees
- moved MOTOR4-C5 2.64 mm to (109.0, 113.5), turned to 180 degrees
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Connections:
- ESP-U1 pad 12: MOTOR4_ISENSE_A -> SDA2
- ESP-U1 pad 17: MOTOR4_ISENSE_B -> SCL2
- ESP-U1 pad 18: VBAT_SENSE -> SDA3
- ESP-U1 pad 19: MOTOR4_FAULT -> SCL3
- ESP-U1 pad 25: MOTOR2_FAULT -> unconnected-(ESP-U1-IO48-Pad25)
- ESP-U1 pad 33: IMU_SDA -> unconnected-(ESP-U1-IO40-Pad33)
- ESP-U1 pad 34: IMU_SCL -> unconnected-(ESP-U1-IO41-Pad34)
- ESP-U1 pad 35: MOTOR3_FAULT -> unconnected-(ESP-U1-IO42-Pad35)
- ESP-U1 pad 36: MOTOR1_FAULT -> MOTOR_FAULT
- ESP-U1 pad 38: MOTOR2_ISENSE_B -> unconnected-(ESP-U1-IO2-Pad38)
- ESP-U1 pad 39: MOTOR2_ISENSE_A -> unconnected-(ESP-U1-IO1-Pad39)
- ESP-U1 pad 4: MOTOR1_ISENSE_A -> SDA0
- ESP-U1 pad 5: MOTOR1_ISENSE_B -> SCL0
- ESP-U1 pad 6: MOTOR3_ISENSE_A -> SDA1
- ESP-U1 pad 7: MOTOR3_ISENSE_B -> SCL1
- IMU-U1 pad 13: IMU_SCL -> SCL0
- IMU-U1 pad 14: IMU_SDA -> SDA0
- MOTOR1-C2 pad 1: MOTOR1_CP -> MOTOR1_VCP
- MOTOR1-C6 pad 1: MOTOR1_AVDD -> MOTOR1_V3P3
- MOTOR1-U1 pad 1: unconnected-(MOTOR1-U1-NC-Pad1) -> MOTOR_ENABLE
- MOTOR1-U1 pad 10: BAT -> MOTOR1_B
- MOTOR1-U1 pad 11: BAT -> MOTOR1_C
- MOTOR1-U1 pad 13: MOTOR1_A -> BAT
- MOTOR1-U1 pad 14: MOTOR1_A -> MOTOR1_VCP
- MOTOR1-U1 pad 16: MOTOR1_B -> BAT
- MOTOR1-U1 pad 17: MOTOR1_B -> unconnected-(MOTOR1-U1-NC-Pad17)
- MOTOR1-U1 pad 18: GND -> MOTOR1_V3P3
- MOTOR1-U1 pad 19: MOTOR1_C -> unconnected-(MOTOR1-U1-NC-Pad19)
- MOTOR1-U1 pad 2: GND -> MOTOR_ENABLE
- MOTOR1-U1 pad 20: MOTOR1_C -> MOTOR_FAULT
- MOTOR1-U1 pad 21: GND -> unconnected-(MOTOR1-U1-NC-Pad21)
- MOTOR1-U1 pad 22: MOTOR1_FAULT -> unconnected-(MOTOR1-U1-NC-Pad22)
- MOTOR1-U1 pad 23: MOTOR_ENABLE -> unconnected-(MOTOR1-U1-NC-Pad23)
- MOTOR1-U1 pad 24: GND -> MOTOR_ENABLE
- MOTOR1-U1 pad 25: MOTOR1_AVDD -> GND
- MOTOR1-U1 pad 3: MOTOR1_BUCK -> MOTOR_ENABLE
- MOTOR1-U1 pad 4: GND -> MOTOR1_PWM_A
- MOTOR1-U1 pad 5: MOTOR1_SW_BK -> MOTOR1_PWM_B
- MOTOR1-U1 pad 6: MOTOR1_CPL -> MOTOR1_PWM_C
- MOTOR1-U1 pad 7: MOTOR1_CPH -> BAT
- MOTOR1-U1 pad 8: MOTOR1_CP -> GND
- MOTOR1-U1 pad 9: BAT -> MOTOR1_A
- MOTOR2-C2 pad 1: MOTOR2_CP -> MOTOR2_VCP
- MOTOR2-C6 pad 1: MOTOR2_AVDD -> MOTOR2_V3P3
- MOTOR2-U1 pad 1: unconnected-(MOTOR2-U1-NC-Pad1) -> MOTOR_ENABLE
- MOTOR2-U1 pad 10: BAT -> MOTOR2_B
- MOTOR2-U1 pad 11: BAT -> MOTOR2_C
- MOTOR2-U1 pad 13: MOTOR2_A -> BAT
- MOTOR2-U1 pad 14: MOTOR2_A -> MOTOR2_VCP
- MOTOR2-U1 pad 16: MOTOR2_B -> BAT
- MOTOR2-U1 pad 17: MOTOR2_B -> unconnected-(MOTOR2-U1-NC-Pad17)
- MOTOR2-U1 pad 18: GND -> MOTOR2_V3P3
- MOTOR2-U1 pad 19: MOTOR2_C -> unconnected-(MOTOR2-U1-NC-Pad19)
- MOTOR2-U1 pad 2: GND -> MOTOR_ENABLE
- MOTOR2-U1 pad 20: MOTOR2_C -> MOTOR_FAULT
- MOTOR2-U1 pad 21: GND -> unconnected-(MOTOR2-U1-NC-Pad21)
- MOTOR2-U1 pad 22: MOTOR2_FAULT -> unconnected-(MOTOR2-U1-NC-Pad22)
- MOTOR2-U1 pad 23: MOTOR_ENABLE -> unconnected-(MOTOR2-U1-NC-Pad23)
- MOTOR2-U1 pad 24: GND -> MOTOR_ENABLE
- MOTOR2-U1 pad 25: MOTOR2_AVDD -> GND
- MOTOR2-U1 pad 3: MOTOR2_BUCK -> MOTOR_ENABLE
- MOTOR2-U1 pad 4: GND -> MOTOR2_PWM_A
- MOTOR2-U1 pad 5: MOTOR2_SW_BK -> MOTOR2_PWM_B
- MOTOR2-U1 pad 6: MOTOR2_CPL -> MOTOR2_PWM_C
- MOTOR2-U1 pad 7: MOTOR2_CPH -> BAT
- MOTOR2-U1 pad 8: MOTOR2_CP -> GND
- MOTOR2-U1 pad 9: BAT -> MOTOR2_A
- MOTOR3-C2 pad 1: MOTOR3_CP -> MOTOR3_VCP
- MOTOR3-C6 pad 1: MOTOR3_AVDD -> MOTOR3_V3P3
- MOTOR3-U1 pad 1: unconnected-(MOTOR3-U1-NC-Pad1) -> MOTOR_ENABLE
- MOTOR3-U1 pad 10: BAT -> MOTOR3_B
- MOTOR3-U1 pad 11: BAT -> MOTOR3_C
- MOTOR3-U1 pad 13: MOTOR3_A -> BAT
- MOTOR3-U1 pad 14: MOTOR3_A -> MOTOR3_VCP
- MOTOR3-U1 pad 16: MOTOR3_B -> BAT
- MOTOR3-U1 pad 17: MOTOR3_B -> unconnected-(MOTOR3-U1-NC-Pad17)
- MOTOR3-U1 pad 18: GND -> MOTOR3_V3P3
- MOTOR3-U1 pad 19: MOTOR3_C -> unconnected-(MOTOR3-U1-NC-Pad19)
- MOTOR3-U1 pad 2: GND -> MOTOR_ENABLE
- MOTOR3-U1 pad 20: MOTOR3_C -> MOTOR_FAULT
- MOTOR3-U1 pad 21: GND -> unconnected-(MOTOR3-U1-NC-Pad21)
- MOTOR3-U1 pad 22: MOTOR3_FAULT -> unconnected-(MOTOR3-U1-NC-Pad22)
- MOTOR3-U1 pad 23: MOTOR_ENABLE -> unconnected-(MOTOR3-U1-NC-Pad23)
- MOTOR3-U1 pad 24: GND -> MOTOR_ENABLE
- MOTOR3-U1 pad 25: MOTOR3_AVDD -> GND
- MOTOR3-U1 pad 3: MOTOR3_BUCK -> MOTOR_ENABLE
- MOTOR3-U1 pad 4: GND -> MOTOR3_PWM_A
- MOTOR3-U1 pad 5: MOTOR3_SW_BK -> MOTOR3_PWM_B
- MOTOR3-U1 pad 6: MOTOR3_CPL -> MOTOR3_PWM_C
- MOTOR3-U1 pad 7: MOTOR3_CPH -> BAT
- MOTOR3-U1 pad 8: MOTOR3_CP -> GND
- MOTOR3-U1 pad 9: BAT -> MOTOR3_A
- MOTOR4-C2 pad 1: MOTOR4_CP -> MOTOR4_VCP
- MOTOR4-C6 pad 1: MOTOR4_AVDD -> MOTOR4_V3P3
- MOTOR4-U1 pad 1: unconnected-(MOTOR4-U1-NC-Pad1) -> MOTOR_ENABLE
- MOTOR4-U1 pad 10: BAT -> MOTOR4_B
- MOTOR4-U1 pad 11: BAT -> MOTOR4_C
- MOTOR4-U1 pad 13: MOTOR4_A -> BAT
- MOTOR4-U1 pad 14: MOTOR4_A -> MOTOR4_VCP
- MOTOR4-U1 pad 16: MOTOR4_B -> BAT
- MOTOR4-U1 pad 17: MOTOR4_B -> unconnected-(MOTOR4-U1-NC-Pad17)
- MOTOR4-U1 pad 18: GND -> MOTOR4_V3P3
- MOTOR4-U1 pad 19: MOTOR4_C -> unconnected-(MOTOR4-U1-NC-Pad19)
- MOTOR4-U1 pad 2: GND -> MOTOR_ENABLE
- MOTOR4-U1 pad 20: MOTOR4_C -> MOTOR_FAULT
- MOTOR4-U1 pad 21: GND -> unconnected-(MOTOR4-U1-NC-Pad21)
- MOTOR4-U1 pad 22: MOTOR4_FAULT -> unconnected-(MOTOR4-U1-NC-Pad22)
- MOTOR4-U1 pad 23: MOTOR_ENABLE -> unconnected-(MOTOR4-U1-NC-Pad23)
- MOTOR4-U1 pad 24: GND -> MOTOR_ENABLE
- MOTOR4-U1 pad 25: MOTOR4_AVDD -> GND
- MOTOR4-U1 pad 3: MOTOR4_BUCK -> MOTOR_ENABLE
- MOTOR4-U1 pad 4: GND -> MOTOR4_PWM_A
- MOTOR4-U1 pad 5: MOTOR4_SW_BK -> MOTOR4_PWM_B
- MOTOR4-U1 pad 6: MOTOR4_CPL -> MOTOR4_PWM_C
- MOTOR4-U1 pad 7: MOTOR4_CPH -> BAT
- MOTOR4-U1 pad 8: MOTOR4_CP -> GND
- MOTOR4-U1 pad 9: BAT -> MOTOR4_A
Routing:
- net MOTOR_FAULT: track 0.00 -> 113.6 mm, vias 0 -> 14
- net SDA0: track 0.00 -> 84.4 mm, vias 0 -> 8
- net MOTOR3_FAULT: track 77.3 -> 0.00 mm, vias 5 -> 0
- net MOTOR3_ISENSE_B_RAW: track 59.7 -> 0.00 mm, vias 3 -> 0
- net SCL1: track 0.00 -> 54.0 mm, vias 0 -> 2
- net SDA1: track 0.00 -> 53.6 mm, vias 0 -> 7
- net SCL0: track 0.00 -> 52.9 mm, vias 0 -> 5
- net SCL2: track 0.00 -> 46.1 mm, vias 0 -> 4
- net MOTOR4_ISENSE_B_RAW: track 45.0 -> 0.00 mm, vias 6 -> 0
- net MOTOR4_FAULT: track 43.7 -> 0.00 mm, vias 5 -> 0
- net V3_3: track 189.1 -> 231.6 mm, vias 14 -> 11
- net MOTOR3_ISENSE_A_RAW: track 41.5 -> 0.00 mm, vias 2 -> 0
- net SCL3: track 0.00 -> 40.8 mm, vias 0 -> 6
- net VIN: track 64.8 -> 24.2 mm, vias 9 -> 2
- net MOTOR4_ISENSE_A_RAW: track 38.2 -> 0.00 mm, vias 2 -> 0
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Other:
- board size 50 x 65 mm -> 50 x 69.5 mm
- board text added: "M1"
- board text added: "M2"
- board text added: "USB"
- board text removed: "bat"
- board text removed: "m1"
- board text removed: "m2"

Commit message: cleanup
Parts:
- ENC-J1: value ENC-J1 -> PZ254V-11-04P
- ENC-J2: value ENC-J2 -> PZ254V-11-04P
- ENC-J3: value ENC-J3 -> PZ254V-11-04P
- ENC-J4: value ENC-J4 -> PZ254V-11-04P
- MOTOR-J1: value WJ2EDGR-5.08-03P-14-00A -> PZ254V-11-03P; footprint ria:WJ2EDGR-5.08-03P-14-00A -> ria:MOTOR-J1
- MOTOR-J2: value WJ2EDGR-5.08-03P-14-00A -> PZ254V-11-03P; footprint ria:WJ2EDGR-5.08-03P-14-00A -> ria:MOTOR-J2
- MOTOR-J3, MOTOR-J4, MOTOR-J5, MOTOR-J6, MOTOR-J7, MOTOR-J8: value GC3510-F -> motor wires
- POWER-J1: value XT60PW-M -> XT60PB-M.G.Y
- moved POWER-J1 1.60 mm to (83.4, 77.3), turned to 0 degrees
Routing:
- net MOTOR2_B: track 16.2 -> 20.0 mm, vias 0 -> 1
- net SCL1: track 54.0 -> 57.3 mm
- net MOTOR2_A: track 13.1 -> 16.1 mm
- net MOTOR1_C: track 15.5 -> 16.3 mm
- net MOTOR1_A: track 28.7 -> 28.1 mm
- net MOTOR2_C: track 22.9 -> 22.4 mm
