File: pcb/ria.kicad_sch (KiCad schematic)
At the start: 104 parts

Commit message: remove obsolete pcb copies and generated documentation
Parts:
- removed ESP-C2: 100nF, ria:ESP-C2, symbol ria:ESP-C2
- removed IMU-R1, IMU-R2: 4.7kΩ, ria:R_0603_1608Metric, symbol ria:MOTOR-RS
- removed MOTOR1-C10, MOTOR2-C10, MOTOR3-C10, MOTOR4-C10, SENSE-C1: 100nF, ria:C_0603_1608Metric, symbol ria:MOTOR1-C2
- removed MOTOR1-C11, MOTOR1-C12, MOTOR2-C11, MOTOR2-C12, MOTOR3-C11, MOTOR3-C12, MOTOR4-C11, MOTOR4-C12: 22pF, ria:C_0603_1608Metric, symbol ria:MOTOR1-C2
- removed MOTOR1-C7, MOTOR2-C7, MOTOR3-C7, MOTOR4-C7: 47nF, ria:C_0603_1608Metric, symbol ria:MOTOR1-C2
- removed MOTOR1-C8, MOTOR2-C8, MOTOR3-C8, MOTOR4-C8: 22uF, ria:C_0805_2012Metric, symbol ria:MOTOR1-C2
- removed MOTOR1-R1, MOTOR2-R1, MOTOR3-R1, MOTOR4-R1: 47kΩ, ria:R_0603_1608Metric, symbol ria:MOTOR-RS
- removed MOTOR1-R2, MOTOR2-R2, MOTOR3-R2, MOTOR4-R2: 22Ω, ria:R_0603_1608Metric, symbol ria:MOTOR-RS
- removed MOTOR1-R3, MOTOR2-R3, MOTOR3-R3, MOTOR4-R3: 5.1kΩ, ria:R_0603_1608Metric, symbol ria:MOTOR-RS
- removed MOTOR1-R4, MOTOR1-R5, MOTOR2-R4, MOTOR2-R5, MOTOR3-R4, MOTOR3-R5, MOTOR4-R4, MOTOR4-R5: 330Ω, ria:R_0603_1608Metric, symbol ria:MOTOR-RS
- removed POWER-C2: 100nF, ria:POWER-C2, symbol ria:POWER-C2
- removed SENSE-R1: 100kΩ, ria:R_0603_1608Metric, symbol ria:MOTOR-RS
- removed SENSE-R2: 20kΩ, ria:R_0603_1608Metric, symbol ria:MOTOR-RS
- removed USB-C1: 100nF, ria:USB-C1, symbol ria:USB-C1
- added ENC-J1: ENC-J1, ria:ENC-J1, symbol ria:ENC-J1
- added ENC-J2: ENC-J2, ria:ENC-J2, symbol ria:ENC-J2
- added ENC-J3: ENC-J3, ria:ENC-J3, symbol ria:ENC-J3
- added ENC-J4: ENC-J4, ria:ENC-J4, symbol ria:ENC-J4
- added ENC-RC0: 4.7kΩ, ria:ENC-RC0, symbol ria:ENC-RC0
- added ENC-RC1: 4.7kΩ, ria:ENC-RC1, symbol ria:ENC-RC1
- added ENC-RC2: 4.7kΩ, ria:ENC-RC2, symbol ria:ENC-RC2
- added ENC-RC3: 4.7kΩ, ria:ENC-RC3, symbol ria:ENC-RC3
- added ENC-RD0: 4.7kΩ, ria:ENC-RD0, symbol ria:ENC-RD0
- added ENC-RD1: 4.7kΩ, ria:ENC-RD1, symbol ria:ENC-RD1
- added ENC-RD2: 4.7kΩ, ria:ENC-RD2, symbol ria:ENC-RD2
- added ENC-RD3: 4.7kΩ, ria:ENC-RD3, symbol ria:ENC-RD3
- added MOTOR-R2: 10kΩ, ria:MOTOR-RS, symbol ria:MOTOR-RS
- ESP-C3: footprint ria:ESP-C3 -> ria:C_0805_2012Metric; LCSC C15849 -> C28323; MPN (none) -> CL21B105KBFNNNE; Manufacturer (none) -> Samsung Electro-Mechanics; Supplier Part Number (none) -> C28323
- MOTOR1-C2: footprint ria:C_0603_1608Metric -> ria:C_0805_2012Metric; LCSC C15849 -> C28323; MPN CL10A105KB8NNNC -> CL21B105KBFNNNE; Supplier Part Number (none) -> C28323
- MOTOR1-C3: footprint ria:C_0603_1608Metric -> ria:MOTOR1-C3; symbol ria:MOTOR1-C2 -> ria:MOTOR1-C3; MPN CC0603KRX7R9BB104 -> (none); Manufacturer YAGEO -> (none)
- MOTOR1-C5: value 10uF -> 22uF; symbol ria:MOTOR1-C2 -> ria:MOTOR1-C5; LCSC C89632 -> C12891; MPN CL31B106KBHNNNE -> CL31A226KAHNNNE; Supplier Part Number (none) -> C12891
- MOTOR1-C6: value 1uF -> 4.7uF; footprint ria:C_0805_2012Metric -> ria:MOTOR1-C6; symbol ria:MOTOR1-C2 -> ria:MOTOR1-C6; LCSC C28323 -> C19666; MPN CL21B105KBFNNNE -> CL10A475KO8NNNC; Manufacturer Samsung Electro-Mechanics -> (none)
- MOTOR1-U1: value DRV8316CTRGFR -> SS6343M-QF-TP; footprint ria:DRV8316CTRGFR -> ria:SS6343M-QF-TP; symbol ria:DRV8316CTRGFR -> ria:MOTOR1-U1; LCSC C6602057 -> C5370899; MPN DRV8316CTRGFR -> SS6343M-QF-TP; Manufacturer Texas Instruments -> (none)
- MOTOR2-C2: footprint ria:C_0603_1608Metric -> ria:C_0805_2012Metric; symbol ria:MOTOR1-C2 -> ria:MOTOR2-C2; LCSC C15849 -> C28323; MPN CL10A105KB8NNNC -> CL21B105KBFNNNE; Supplier Part Number (none) -> C28323
- MOTOR2-C3: footprint ria:C_0603_1608Metric -> ria:MOTOR2-C3; symbol ria:MOTOR1-C2 -> ria:MOTOR2-C3; MPN CC0603KRX7R9BB104 -> (none); Manufacturer YAGEO -> (none)
- MOTOR2-C5: value 10uF -> 22uF; symbol ria:MOTOR1-C2 -> ria:MOTOR2-C5; LCSC C89632 -> C12891; MPN CL31B106KBHNNNE -> CL31A226KAHNNNE; Supplier Part Number (none) -> C12891
- MOTOR2-C6: value 1uF -> 4.7uF; footprint ria:C_0805_2012Metric -> ria:MOTOR2-C6; symbol ria:MOTOR1-C2 -> ria:MOTOR2-C6; LCSC C28323 -> C19666; MPN CL21B105KBFNNNE -> CL10A475KO8NNNC; Manufacturer Samsung Electro-Mechanics -> (none)
- MOTOR2-U1: value DRV8316CTRGFR -> SS6343M-QF-TP; footprint ria:DRV8316CTRGFR -> ria:SS6343M-QF-TP; symbol ria:DRV8316CTRGFR -> ria:MOTOR2-U1; LCSC C6602057 -> C5370899; MPN DRV8316CTRGFR -> SS6343M-QF-TP; Manufacturer Texas Instruments -> (none)
- MOTOR3-C2: footprint ria:C_0603_1608Metric -> ria:C_0805_2012Metric; symbol ria:MOTOR1-C2 -> ria:MOTOR3-C2; LCSC C15849 -> C28323; MPN CL10A105KB8NNNC -> CL21B105KBFNNNE; Supplier Part Number (none) -> C28323
- MOTOR3-C3: footprint ria:C_0603_1608Metric -> ria:MOTOR3-C3; symbol ria:MOTOR1-C2 -> ria:MOTOR3-C3; MPN CC0603KRX7R9BB104 -> (none); Manufacturer YAGEO -> (none)
- MOTOR3-C5: value 10uF -> 22uF; symbol ria:MOTOR1-C2 -> ria:MOTOR3-C5; LCSC C89632 -> C12891; MPN CL31B106KBHNNNE -> CL31A226KAHNNNE; Supplier Part Number (none) -> C12891
- MOTOR3-C6: value 1uF -> 4.7uF; footprint ria:C_0805_2012Metric -> ria:MOTOR3-C6; symbol ria:MOTOR1-C2 -> ria:MOTOR3-C6; LCSC C28323 -> C19666; MPN CL21B105KBFNNNE -> CL10A475KO8NNNC; Manufacturer Samsung Electro-Mechanics -> (none)
- MOTOR3-U1: value DRV8316CTRGFR -> SS6343M-QF-TP; footprint ria:DRV8316CTRGFR -> ria:SS6343M-QF-TP; symbol ria:DRV8316CTRGFR -> ria:MOTOR3-U1; LCSC C6602057 -> C5370899; MPN DRV8316CTRGFR -> SS6343M-QF-TP; Manufacturer Texas Instruments -> (none)
- MOTOR4-C2: footprint ria:C_0603_1608Metric -> ria:C_0805_2012Metric; symbol ria:MOTOR1-C2 -> ria:MOTOR4-C2; LCSC C15849 -> C28323; MPN CL10A105KB8NNNC -> CL21B105KBFNNNE; Supplier Part Number (none) -> C28323
- MOTOR4-C3: footprint ria:C_0603_1608Metric -> ria:MOTOR4-C3; symbol ria:MOTOR1-C2 -> ria:MOTOR4-C3; MPN CC0603KRX7R9BB104 -> (none); Manufacturer YAGEO -> (none)
- MOTOR4-C5: value 10uF -> 22uF; symbol ria:MOTOR1-C2 -> ria:MOTOR4-C5; LCSC C89632 -> C12891; MPN CL31B106KBHNNNE -> CL31A226KAHNNNE; Supplier Part Number (none) -> C12891
- MOTOR4-C6: value 1uF -> 4.7uF; footprint ria:C_0805_2012Metric -> ria:MOTOR4-C6; symbol ria:MOTOR1-C2 -> ria:MOTOR4-C6; LCSC C28323 -> C19666; MPN CL21B105KBFNNNE -> CL10A475KO8NNNC; Manufacturer Samsung Electro-Mechanics -> (none)
- MOTOR4-U1: value DRV8316CTRGFR -> SS6343M-QF-TP; footprint ria:DRV8316CTRGFR -> ria:SS6343M-QF-TP; symbol ria:DRV8316CTRGFR -> ria:MOTOR4-U1; LCSC C6602057 -> C5370899; MPN DRV8316CTRGFR -> SS6343M-QF-TP; Manufacturer Texas Instruments -> (none)
- POWER-J1: value XT60PB-M.G.Y -> XT60PW-M; LCSC C19268037 -> C98732; MPN XT60PB-M.G.Y -> XT60PW-M
- POWER-U1: value AP63300WU-7 -> AP63301WU-7; LCSC C2158012 -> C2158003; MPN AP63300WU-7 -> AP63301WU-7; Manufacturer (none) -> Diodes Incorporated; Supplier Part Number (none) -> C2158003
Connections:
- net MOTOR1_BUCK is gone; now on net MOTOR_ENABLE: MOTOR1-U1.3 (ENC)
- net MOTOR1_CPH is gone; now on net BAT: MOTOR1-U1.7 (VIN)
- net MOTOR1_CPL is gone; now on net MOTOR1_PWM_C: MOTOR1-U1.6 (PWMC)
- net MOTOR1_SW_BK is gone; now on net MOTOR1_PWM_B: MOTOR1-U1.5 (PWMB)
- net MOTOR2_BUCK is gone; now on net MOTOR_ENABLE: MOTOR2-U1.3 (ENC)
- net MOTOR2_CPH is gone; now on net BAT: MOTOR2-U1.7 (VIN)
- net MOTOR2_CPL is gone; now on net MOTOR2_PWM_C: MOTOR2-U1.6 (PWMC)
- net MOTOR2_SW_BK is gone; now on net MOTOR2_PWM_B: MOTOR2-U1.5 (PWMB)
- net MOTOR3_BUCK is gone; now on net MOTOR_ENABLE: MOTOR3-U1.3 (ENC)
- net MOTOR3_CPH is gone; now on net BAT: MOTOR3-U1.7 (VIN)
- net MOTOR3_CPL is gone; now on net MOTOR3_PWM_C: MOTOR3-U1.6 (PWMC)
- net MOTOR3_SW_BK is gone; now on net MOTOR3_PWM_B: MOTOR3-U1.5 (PWMB)
- net MOTOR4_BUCK is gone; now on net MOTOR_ENABLE: MOTOR4-U1.3 (ENC)
- net MOTOR4_CPH is gone; now on net BAT: MOTOR4-U1.7 (VIN)
- net MOTOR4_CPL is gone; now on net MOTOR4_PWM_C: MOTOR4-U1.6 (PWMC)
- net MOTOR4_SW_BK is gone; now on net MOTOR4_PWM_B: MOTOR4-U1.5 (PWMB)
- net BAT: now also MOTOR1-U1.13 (VIN), MOTOR1-U1.16 (VIN_LDO), MOTOR2-U1.13 (VIN), MOTOR2-U1.16 (VIN_LDO), MOTOR3-U1.13 (VIN), MOTOR3-U1.16 (VIN_LDO), MOTOR4-U1.13 (VIN), MOTOR4-U1.16 (VIN_LDO); no longer MOTOR1-U1.10 (VM_2), MOTOR1-U1.11 (VM_3), MOTOR1-U1.9 (VM_1), MOTOR2-U1.10 (VM_2), MOTOR2-U1.11 (VM_3), MOTOR2-U1.9 (VM_1), MOTOR3-U1.10 (VM_2), MOTOR3-U1.11 (VM_3), MOTOR3-U1.9 (VM_1), MOTOR4-U1.10 (VM_2), MOTOR4-U1.11 (VM_3), MOTOR4-U1.9 (VM_1)
- net GND: now also MOTOR1-U1.25 (EP), MOTOR1-U1.8 (LSS), MOTOR2-U1.25 (EP), MOTOR2-U1.8 (LSS), MOTOR3-U1.25 (EP), MOTOR3-U1.8 (LSS), MOTOR4-U1.25 (EP), MOTOR4-U1.8 (LSS), ENC-J1.2, ENC-J2.2, ENC-J3.2, ENC-J4.2; no longer MOTOR1-U1.18 (PGND_3), MOTOR1-U1.2 (AGND_1), MOTOR1-U1.21 (DRVOFF), MOTOR1-U1.24 (VSEL_BK), MOTOR1-U1.26 (AGND_2), MOTOR1-U1.34 (SLEW), MOTOR1-U1.35 (OCP/SR), MOTOR1-U1.4 (GND_BK), MOTOR1-U1.41 (GND), MOTOR2-U1.18 (PGND_3), MOTOR2-U1.2 (AGND_1), MOTOR2-U1.21 (DRVOFF), MOTOR2-U1.24 (VSEL_BK), MOTOR2-U1.26 (AGND_2), MOTOR2-U1.34 (SLEW), MOTOR2-U1.35 (OCP/SR), MOTOR2-U1.4 (GND_BK), MOTOR2-U1.41 (GND), MOTOR3-U1.18 (PGND_3), MOTOR3-U1.2 (AGND_1), MOTOR3-U1.21 (DRVOFF), MOTOR3-U1.24 (VSEL_BK), MOTOR3-U1.26 (AGND_2), MOTOR3-U1.34 (SLEW), MOTOR3-U1.35 (OCP/SR), MOTOR3-U1.4 (GND_BK), MOTOR3-U1.41 (GND), MOTOR4-U1.18 (PGND_3), MOTOR4-U1.2 (AGND_1), MOTOR4-U1.21 (DRVOFF), MOTOR4-U1.24 (VSEL_BK), MOTOR4-U1.26 (AGND_2), MOTOR4-U1.34 (SLEW), MOTOR4-U1.35 (OCP/SR), MOTOR4-U1.4 (GND_BK), MOTOR4-U1.41 (GND)
- net MOTOR1_A: now also MOTOR1-U1.9 (SA); no longer MOTOR1-U1.13 (OUTA_1), MOTOR1-U1.14 (OUTA_2)
- net MOTOR1_B: now also MOTOR1-U1.10 (SB); no longer MOTOR1-U1.16 (OUTB_1), MOTOR1-U1.17 (OUTB_2)
- net MOTOR1_C: now also MOTOR1-U1.11 (SC); no longer MOTOR1-U1.19 (OUTC_1), MOTOR1-U1.20 (OUTC_2)
- net MOTOR1_PWM_A: now also MOTOR1-U1.4 (PWMA); no longer MOTOR1-U1.27 (INHA)
- net MOTOR1_PWM_B: no longer MOTOR1-U1.29 (INHB)
- net MOTOR1_PWM_C: no longer MOTOR1-U1.31 (INHC)
- net MOTOR2_A: now also MOTOR2-U1.9 (SA); no longer MOTOR2-U1.13 (OUTA_1), MOTOR2-U1.14 (OUTA_2)
- net MOTOR2_B: now also MOTOR2-U1.10 (SB); no longer MOTOR2-U1.16 (OUTB_1), MOTOR2-U1.17 (OUTB_2)
- net MOTOR2_C: now also MOTOR2-U1.11 (SC); no longer MOTOR2-U1.19 (OUTC_1), MOTOR2-U1.20 (OUTC_2)
- net MOTOR2_PWM_A: now also MOTOR2-U1.4 (PWMA); no longer MOTOR2-U1.27 (INHA)
- net MOTOR2_PWM_B: no longer MOTOR2-U1.29 (INHB)
- net MOTOR2_PWM_C: no longer MOTOR2-U1.31 (INHC)
- net MOTOR3_A: now also MOTOR3-U1.9 (SA); no longer MOTOR3-U1.13 (OUTA_1), MOTOR3-U1.14 (OUTA_2)
- net MOTOR3_B: now also MOTOR3-U1.10 (SB); no longer MOTOR3-U1.16 (OUTB_1), MOTOR3-U1.17 (OUTB_2)
- net MOTOR3_C: now also MOTOR3-U1.11 (SC); no longer MOTOR3-U1.19 (OUTC_1), MOTOR3-U1.20 (OUTC_2)
- net MOTOR3_PWM_A: now also MOTOR3-U1.4 (PWMA); no longer MOTOR3-U1.27 (INHA)
- net MOTOR3_PWM_B: no longer MOTOR3-U1.29 (INHB)
- net MOTOR3_PWM_C: no longer MOTOR3-U1.31 (INHC)
- net MOTOR4_A: now also MOTOR4-U1.9 (SA); no longer MOTOR4-U1.13 (OUTA_1), MOTOR4-U1.14 (OUTA_2)
- net MOTOR4_B: now also MOTOR4-U1.10 (SB); no longer MOTOR4-U1.16 (OUTB_1), MOTOR4-U1.17 (OUTB_2)
- net MOTOR4_C: now also MOTOR4-U1.11 (SC); no longer MOTOR4-U1.19 (OUTC_1), MOTOR4-U1.20 (OUTC_2)
- net MOTOR4_PWM_A: now also MOTOR4-U1.4 (PWMA); no longer MOTOR4-U1.27 (INHA)
- net MOTOR4_PWM_B: no longer MOTOR4-U1.29 (INHB)
- net MOTOR4_PWM_C: no longer MOTOR4-U1.31 (INHC)
- net MOTOR_ENABLE: now also MOTOR1-U1.1 (ENA), MOTOR1-U1.2 (ENB), MOTOR1-U1.24 (nSLEEP), MOTOR2-U1.1 (ENA), MOTOR2-U1.2 (ENB), MOTOR2-U1.24 (nSLEEP), MOTOR3-U1.1 (ENA), MOTOR3-U1.2 (ENB), MOTOR3-U1.24 (nSLEEP), MOTOR4-U1.1 (ENA), MOTOR4-U1.2 (ENB), MOTOR4-U1.24 (nSLEEP); no longer MOTOR1-U1.23 (NSLEEP), MOTOR2-U1.23 (NSLEEP), MOTOR3-U1.23 (NSLEEP), MOTOR4-U1.23 (NSLEEP)
- net V3_3: now also ENC-J1.1, ENC-J2.1, ENC-J3.1, ENC-J4.1, ENC-RC0.1, ENC-RC1.1, ENC-RC2.1, ENC-RC3.1, ENC-RD0.1, ENC-RD1.1, ENC-RD2.1, ENC-RD3.1, MOTOR-R2.1
- net IMU_SCL: no longer names the net of ESP-U1.34 (IO41)
- net IMU_SCL: no longer IMU-U1.13 (SCK)
- net IMU_SDA: no longer names the net of ESP-U1.33 (IO40)
- net IMU_SDA: no longer IMU-U1.14 (SDA)
- removed net MOTOR1_AVDD: MOTOR1-C6.1, MOTOR1-U1.25 (AVDD), MOTOR1-U1.28 (INLA), MOTOR1-U1.30 (INLB), MOTOR1-U1.32 (INLC), MOTOR1-U1.37 (VREF/_ILIM)
- net MOTOR1_CP renamed MOTOR1_VCP
- net MOTOR1_VCP: now also MOTOR1-U1.14 (VCP); no longer MOTOR1-U1.8 (CP)
- net MOTOR1_FAULT: no longer names the net of MOTOR1-U1.22 (NC)
- net MOTOR1_FAULT: no longer ESP-U1.36 (RXD0)
- net MOTOR1_ISENSE_A renamed SDA0
- net SDA0: now also IMU-U1.14 (SDA), ENC-J1.3, ENC-RD0.2
- removed net MOTOR1_ISENSE_A_RAW: MOTOR1-U1.40 (SOA)
- net MOTOR1_ISENSE_B renamed SCL0
- net SCL0: now also IMU-U1.13 (SCK), ENC-J1.4, ENC-RC0.2
- removed net MOTOR1_ISENSE_B_RAW: MOTOR1-U1.39 (SOB)
- removed net MOTOR1_MODE: MOTOR1-U1.33 (MODE)
- removed net MOTOR2_AVDD: MOTOR2-C6.1, MOTOR2-U1.25 (AVDD), MOTOR2-U1.28 (INLA), MOTOR2-U1.30 (INLB), MOTOR2-U1.32 (INLC), MOTOR2-U1.37 (VREF/_ILIM)
- net MOTOR2_CP renamed MOTOR2_VCP
- net MOTOR2_VCP: now also MOTOR2-U1.14 (VCP); no longer MOTOR2-U1.8 (CP)
- net MOTOR2_FAULT: no longer names the net of MOTOR2-U1.22 (NC)
- net MOTOR2_FAULT: no longer ESP-U1.25 (IO48)
- net MOTOR2_ISENSE_A: no longer names the net of ESP-U1.39 (IO1)
- removed net MOTOR2_ISENSE_A_RAW: MOTOR2-U1.40 (SOA)
- net MOTOR2_ISENSE_B: no longer names the net of ESP-U1.38 (IO2)
- removed net MOTOR2_ISENSE_B_RAW: MOTOR2-U1.39 (SOB)
- removed net MOTOR2_MODE: MOTOR2-U1.33 (MODE)
- removed net MOTOR3_AVDD: MOTOR3-C6.1, MOTOR3-U1.25 (AVDD), MOTOR3-U1.28 (INLA), MOTOR3-U1.30 (INLB), MOTOR3-U1.32 (INLC), MOTOR3-U1.37 (VREF/_ILIM)
- net MOTOR3_CP renamed MOTOR3_VCP
- net MOTOR3_VCP: now also MOTOR3-U1.14 (VCP); no longer MOTOR3-U1.8 (CP)
- net MOTOR3_FAULT: no longer names the net of MOTOR3-U1.22 (NC)
- net MOTOR3_FAULT: no longer ESP-U1.35 (IO42)
- net MOTOR3_ISENSE_A renamed SDA1
- net SDA1: now also ENC-J2.3, ENC-RD1.2
- removed net MOTOR3_ISENSE_A_RAW: MOTOR3-U1.40 (SOA)
- net MOTOR3_ISENSE_B renamed SCL1
- net SCL1: now also ENC-J2.4, ENC-RC1.2
- removed net MOTOR3_ISENSE_B_RAW: MOTOR3-U1.39 (SOB)
- removed net MOTOR3_MODE: MOTOR3-U1.33 (MODE)
- removed net MOTOR4_AVDD: MOTOR4-C6.1, MOTOR4-U1.25 (AVDD), MOTOR4-U1.28 (INLA), MOTOR4-U1.30 (INLB), MOTOR4-U1.32 (INLC), MOTOR4-U1.37 (VREF/_ILIM)
- net MOTOR4_CP renamed MOTOR4_VCP
- net MOTOR4_VCP: now also MOTOR4-U1.14 (VCP); no longer MOTOR4-U1.8 (CP)
- net MOTOR4_FAULT: no longer names the net of MOTOR4-U1.22 (NC)
- net MOTOR4_FAULT: no longer ESP-U1.19 (IO11)
- net MOTOR4_ISENSE_A renamed SDA2
- net SDA2: now also ENC-J3.3, ENC-RD2.2
- removed net MOTOR4_ISENSE_A_RAW: MOTOR4-U1.40 (SOA)
- net MOTOR4_ISENSE_B renamed SCL2
- net SCL2: now also ENC-J3.4, ENC-RC2.2
- removed net MOTOR4_ISENSE_B_RAW: MOTOR4-U1.39 (SOB)
- removed net MOTOR4_MODE: MOTOR4-U1.33 (MODE)
- net VBAT_SENSE renamed SDA3
- net SDA3: now also ENC-J4.3, ENC-RD3.2
- new net MOTOR1_V3P3: MOTOR1-C6.1, MOTOR1-U1.18 (V3P3)
- new net MOTOR2_V3P3: MOTOR2-C6.1, MOTOR2-U1.18 (V3P3)
- new net MOTOR3_V3P3: MOTOR3-C6.1, MOTOR3-U1.18 (V3P3)
- new net MOTOR4_V3P3: MOTOR4-C6.1, MOTOR4-U1.18 (V3P3)
- new net MOTOR_FAULT: ESP-U1.36 (RXD0), MOTOR-R2.2, MOTOR1-U1.20 (nFAULT), MOTOR2-U1.20 (nFAULT), MOTOR3-U1.20 (nFAULT), MOTOR4-U1.20 (nFAULT)
- new net SCL3: ENC-J4.4, ENC-RC3.2, ESP-U1.19 (IO11)
- no-connect marks 21 -> 37
Other:
- note added: "enc"
- note removed: "current sensing / battery voltage"
- moved on the sheet: MOTOR-J1, MOTOR-J2, MOTOR-J3, MOTOR-J4, MOTOR-J5, MOTOR-J6, MOTOR-J7, MOTOR-J8, MOTOR1-C2, MOTOR1-C3, MOTOR1-C5, MOTOR1-C6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

Commit message: cleanup
Parts:
- ENC-J1: value ENC-J1 -> PZ254V-11-04P; 3D Model Note (none) -> dimensioned reference model from xfcn pz254v-11 drawing; sq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; MPN (none) -> PZ254V-11-04P; Manufacturer (none) -> XFCN; Supplier (none) -> LCSC; Supplier Part Number (none) -> C2691448
- ENC-J2: value ENC-J2 -> PZ254V-11-04P; 3D Model Note (none) -> dimensioned reference model from xfcn pz254v-11 drawing; sq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; MPN (none) -> PZ254V-11-04P; Manufacturer (none) -> XFCN; Supplier (none) -> LCSC; Supplier Part Number (none) -> C2691448
- ENC-J3: value ENC-J3 -> PZ254V-11-04P; 3D Model Note (none) -> dimensioned reference model from xfcn pz254v-11 drawing; sq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; MPN (none) -> PZ254V-11-04P; Manufacturer (none) -> XFCN; Supplier (none) -> LCSC; Supplier Part Number (none) -> C2691448
- ENC-J4: value ENC-J4 -> PZ254V-11-04P; 3D Model Note (none) -> dimensioned reference model from xfcn pz254v-11 drawing; sq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; MPN (none) -> PZ254V-11-04P; Manufacturer (none) -> XFCN; Supplier (none) -> LCSC; Supplier Part Number (none) -> C2691448
- MOTOR-J1: value WJ2EDGR-5.08-03P-14-00A -> PZ254V-11-03P; footprint ria:WJ2EDGR-5.08-03P-14-00A -> ria:MOTOR-J1; 3D Model Note (none) -> dimensioned reference model from xfcn pz254v-11 drawing; sq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; LCSC C70914 -> C2937625; LCSC Part C70914 -> (none); MPN WJ2EDGR-5.08-03P-14-00A -> PZ254V-11-03P; Manufacturer Ningbo Kangnex Elec -> XFCN; Supplier Part Number C70914 -> C2937625
- MOTOR-J2: value WJ2EDGR-5.08-03P-14-00A -> PZ254V-11-03P; footprint ria:WJ2EDGR-5.08-03P-14-00A -> ria:MOTOR-J2; 3D Model Note (none) -> dimensioned reference model from xfcn pz254v-11 drawing; sq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; LCSC C70914 -> C2937625; LCSC Part C70914 -> (none); MPN WJ2EDGR-5.08-03P-14-00A -> PZ254V-11-03P; Manufacturer Ningbo Kangnex Elec -> XFCN; Supplier Part Number C70914 -> C2937625
- MOTOR-J3, MOTOR-J4, MOTOR-J5, MOTOR-J6, MOTOR-J7, MOTOR-J8: value GC3510-F -> motor wires; LCSC C964714 -> (none); MPN GC3510-F -> (none); now left out of the parts list
- POWER-J1: value XT60PW-M -> XT60PB-M.G.Y; LCSC C98732 -> C19268037; MPN XT60PW-M -> XT60PB-M.G.Y
Connections:
- no-connect marks 37 -> 35
